File: DPB-PCB.kicad_sch (KiCad schematic)
At the start: 15 parts, among them U1 ESP32-S3-WROOM-1-N4R2

Commit message: On production | V0.1
Parts:
- H1, H2, H3, H4: now left out of the parts list
Other:
- added sheet IMU (imu.kicad_sch)
Changed lines of the file:
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@@
     (fill (type none))
   )
-  (rectangle (start 13.97 13.97) (end 180.34 48.26)
+  (rectangle (start 13.97 13.97) (end 209.55 48.26)
     (stroke (width 0) (type dash))
     (fill (type none))
@@
   )
   (symbol (lib_id "Mechanical:MountingHole") (at 265.43 27.94 0) (unit 1)
-    (in_bom yes) (on_board yes) (dnp no) (fields_autoplaced)
+    (in_bom no) (on_board yes) (dnp no) (fields_autoplaced)
     (property "Reference" "H3" (at 267.97 27.305 0)
       (effects (font (size 1.27 1.27)) (justify left))
@@
   )
   (symbol (lib_id "Mechanical:MountingHole") (at 252.73 36.83 0) (unit 1)
-    (in_bom yes) (on_board yes) (dnp no) (fields_autoplaced)
+    (in_bom no) (on_board yes) (dnp no) (fields_autoplaced)
     (property "Reference" "H2" (at 255.27 36.195 0)
       (effects (font (size 1.27 1.27)) (justify left))
@@
   )
   (symbol (lib_id "Mechanical:MountingHole") (at 265.43 36.83 0) (unit 1)
-    (in_bom yes) (on_board yes) (dnp no) (fields_autoplaced)
+    (in_bom no) (on_board yes) (dnp no) (fields_autoplaced)
     (property "Reference" "H4" (at 267.97 36.195 0)
       (effects (font (size 1.27 1.27)) (justify left))
@@
   )
   (symbol (lib_id "Mechanical:MountingHole") (at 252.73 27.94 0) (unit 1)
-    (in_bom yes) (on_board yes) (dnp no) (fields_autoplaced)
+    (in_bom no) (on_board yes) (dnp no) (fields_autoplaced)
     (property "Reference" "H1" (at 255.27 27.305 0)
       (effects (font (size 1.27 1.27)) (justify left))
@@
       )
     )
+  )
+  (sheet (at 180.34 26.67) (size 12.7 12.7) (fields_autoplaced)
+    (stroke (width 0.1524) (type solid))
+    (fill (color 0 0 0 0.0000))
+    (property "Sheetname" "IMU" (at 180.34 25.9584 0)
+      (effects (font (size 1.27 1.27)) (justify left bottom))
+    )
+    (property "Sheetfile" "imu.kicad_sch" (at 180.34 39.9546 0)
+      (effects (font (size 1.27 1.27)) (justify left top))
+    )
+    (instances
+      (project "DPB-PCB"
+        (path "/0a09ce58-c923-4e96-b56b-0b86aca559ed" (page "7"))
+      )
+    )

Commit message: Add hysteresis to IR sensor. Update README file.
Parts:
- C2: footprint Capacitor_SMD:C_01005_0402Metric -> Capacitor_SMD:C_0402_1005Metric
Changed lines of the file:
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@@
       (effects (font (size 1.27 1.27)) (justify left))
     )
-    (property "Footprint" "Capacitor_SMD:C_01005_0402Metric" (at 173.6852 80.01 0)
+    (property "Footprint" "Capacitor_SMD:C_0402_1005Metric" (at 173.6852 80.01 0)
       (effects (font (size 1.27 1.27)) hide)
     )
