File: USB_OTG_connections.kicad_sch (KiCad schematic)
At the start: 5 parts, among them J7 USB_C_OTG, U9 USBLC6-4SC6

Commit message: Add hysteresis to IR sensor. Update README file.
Parts:
- C2: footprint Capacitor_SMD:C_01005_0402Metric -> Capacitor_SMD:C_0402_1005Metric
Changed lines of the file:
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@@
       (effects (font (size 1.27 1.27)) (justify left))
     )
-    (property "Footprint" "Capacitor_SMD:C_01005_0402Metric" (at 153.3652 48.26 0)
+    (property "Footprint" "Capacitor_SMD:C_0402_1005Metric" (at 153.3652 48.26 0)
       (effects (font (size 1.27 1.27)) hide)
     )
