File: USB_connections.kicad_sch (KiCad schematic)
At the start: 21 parts, among them P1 USB_C_Prog, Q3 MMBT5551, Q4 MMBT5551, U2 CP2102N-Axx-xQFN28, U9 USBLC6-4SC6

Commit message: DPB mainboard_v1 completed
Parts:
- removed P1: USB_C_Prog, Connector_USB:USB_C_Receptacle_Molex_105450-0101, symbol Connector:USB_C_Plug
- added C2: 100n 50V, Capacitor_SMD:C_01005_0402Metric, symbol Device:C
- added J1: USB_C_Prog, Connector_USB:USB_C_Receptacle_G-Switch_GT-USB-7010ASV, symbol Connector:USB_C_Receptacle_USB2.0
- added R3 (x2): 10, Resistor_SMD:R_0402_1005Metric, symbol Device:R
- C6: value 10u 50V -> 10u 6V3; footprint Capacitor_SMD:C_1206_3216Metric -> Capacitor_SMD:C_0402_1005Metric; LCSC C13585 -> C15525
- renumbered D4 to D7, D1 to D8, Q3 to Q2, Q4 to Q3, U9 to U4
Connections:
- net COM_D+ is gone; now on net D+: U2.4 (D+), U4.1 (I/O1)
- net D+: now also J1.A6 (D+), J1.B6 (D+); no longer U4.3 (I/O2)
- net D-: now also U2.5 (D-), U4.3 (I/O2), J1.A7 (D-), J1.B7 (D-); no longer U4.6 (I/O4)
- net GND: now also C2.2, J1.A1 (GND), J1.A12 (GND), J1.B1 (GND), J1.B12 (GND)
- net UART_RX: now also R3.2; no longer U2.25 (RXD)
- net UART_TX: now also R3.2; no longer U2.26 (TXD)
- net VBUS: now also C2.1, J1.A4 (VBUS), J1.A9 (VBUS), J1.B4 (VBUS), J1.B9 (VBUS)
- net at R5.1: now also J1.B5 (CC2)
- net at R5.1: now also J1.A5 (CC1)
- net COM_D-: no longer names the net of U4.4 (I/O3)
- net COM_D-: no longer U2.5 (D-)
- new net RXD: R3.1, U2.25 (RXD)
- new net TXD: R3.1, U2.26 (TXD)
- no-connect marks 25 -> 19
Other:
- moved on the sheet: Q2, Q3, R3, R5, U4

Commit message: Add hysteresis to IR sensor. Update README file.
Parts:
- C2: footprint Capacitor_SMD:C_01005_0402Metric -> Capacitor_SMD:C_0402_1005Metric
Changed lines of the file:
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@@
       (effects (font (size 1.27 1.27)) (justify left))
     )
-    (property "Footprint" "Capacitor_SMD:C_01005_0402Metric" (at 186.3852 80.645 0)
+    (property "Footprint" "Capacitor_SMD:C_0402_1005Metric" (at 186.3852 80.645 0)
       (effects (font (size 1.27 1.27)) hide)
     )
@@
       (effects (font (size 1.27 1.27)) (justify left))
     )
-    (property "Footprint" "Capacitor_SMD:C_01005_0402Metric" (at 153.3652 48.26 0)
-      (effects (font (size 1.27 1.27)) hide)
-    )
+    (property "Footprint" "Capacitor_SMD:C_0402_1005Metric" (at 153.3652 48.26 0)
+      (effects (font (size 1.27 1.27)) hide)
+    )
